File: Projeto Kicad/Projeto Kicad/Projeto Kicad.sch (KiCad schematic (older format))
At the start: 10 parts, among them J1 Conn_01x01_Male, J2 Conn_01x01_Male, J3 Conn_01x01_Male, J4 Conn_01x01_Male

Commit message: Finalizado o projeto Kicad
Parts:
- R1: value R_Small -> 360
- pot: value R_POT -> 10k
Connections:
- net +5V: now also lcd.2 (VDD), pot.3; no longer lcd.1 (VSS), pot.1
- net GND: now also lcd.1 (VSS), pot.1; no longer lcd.2 (VDD), pot.3
Changed lines of the file:
@@
 lcd_en
-$Comp
-L power:+5V #PWR?
-U 1 1 6076BEB2
-P 2550 2200
-F 0 "#PWR?" H 2550 2050 50  0001 C CNN
-F 1 "+5V" H 2565 2373 50  0000 C CNN
-F 2 "" H 2550 2200 50  0001 C CNN
-F 3 "" H 2550 2200 50  0001 C CNN
-	1    2550 2200
-	1    0    0    -1
-$EndComp
-Wire Wire Line
-	2550 2200 2550 2600
-$Comp
-L power:GND #PWR?
-U 1 1 6076DE2A
-P 2550 4350
-F 0 "#PWR?" H 2550 4100 50  0001 C CNN
-F 1 "GND" H 2555 4177 50  0000 C CNN
-F 2 "" H 2550 4350 50  0001 C CNN
-F 3 "" H 2550 4350 50  0001 C CNN
-	1    2550 4350
-	1    0    0    -1
-$EndComp
-Wire Wire Line
-	2550 4350 2550 4250
 $Comp
 L Device:R_POT pot
 U 1 1 6076F9A4
 P 1250 4000
-F 0 "pot" H 1181 4046 50  0000 R CNN
-F 1 "R_POT" H 1181 3955 50  0000 R CNN
+F 0 "pot" H 1180 4046 50  0000 R CNN
+F 1 "10k" H 1180 3955 50  0000 R CNN
 F 2 "" H 1250 4000 50  0001 C CNN
 F 3 "~" H 1250 4000 50  0001 C CNN
@@
 	1    0    0    -1
 $EndComp
-Connection ~ 2550 4250
-Wire Wire Line
-	2550 4250 2550 4200
-$Comp
-L power:GND #PWR?
-U 1 1 60773422
-P 2100 3250
-F 0 "#PWR?" H 2100 3000 50  0001 C CNN
-F 1 "GND" H 2105 3077 50  0000 C CNN
-F 2 "" H 2100 3250 50  0001 C CNN
-F 3 "" H 2100 3250 50  0001 C CNN
-	1    2100 3250
-	1    0    0    -1
-$EndComp
 Wire Wire Line
 	1400 4000 2150 4000
-Wire Wire Line
-	1250 4250 1250 4150
-Wire Wire Line
-	1250 4250 2550 4250
-$Comp
-L power:+5V #PWR?
-U 1 1 6077A4FB
-P 1250 3550
-F 0 "#PWR?" H 1250 3400 50  0001 C CNN
-F 1 "+5V" H 1265 3723 50  0000 C CNN
-F 2 "" H 1250 3550 50  0001 C CNN
-F 3 "" H 1250 3550 50  0001 C CNN
-	1    1250 3550
-	1    0    0    -1
-$EndComp
-Wire Wire Line
-	1250 3550 1250 3700
 $Comp
 L Device:R_Small R1
@@
 P 1550 3700
 F 0 "R1" V 1354 3700 50  0000 C CNN
-F 1 "R_Small" V 1445 3700 50  0000 C CNN
+F 1 "360" V 1445 3700 50  0000 C CNN
 F 2 "" H 1550 3700 50  0001 C CNN
 F 3 "~" H 1550 3700 50  0001 C CNN
@@
 	1650 3700 2150 3700
 Wire Wire Line
-	1450 3700 1250 3700
-Connection ~ 1250 3700
-Wire Wire Line
-	1250 3700 1250 3850
-Wire Wire Line
-	2150 3600 1900 3600
-Wire Wire Line
-	1900 3600 1900 3200
-Wire Wire Line
-	1900 3200 2100 3200
-Wire Wire Line
-	2100 3200 2100 3250
-Wire Wire Line
 	6700 4200 6700 3450
 Wire Wire Line
@@
 Wire Wire Line
 	5650 3350 6800 3350
+$Comp
+L power:GND #PWR?
+U 1 1 6079AA64
+P 1650 3200
+F 0 "#PWR?" H 1650 2950 50  0001 C CNN
+F 1 "GND" H 1655 3027 50  0000 C CNN
+F 2 "" H 1650 3200 50  0001 C CNN
+F 3 "" H 1650 3200 50  0001 C CNN
+	1    1650 3200
+	1    0    0    -1
+$EndComp
+Wire Wire Line
+	2550 2600 2550 2500
+Wire Wire Line
+	1900 3600 1900 3150
+Wire Wire Line
+	1900 3150 1650 3150
+Wire Wire Line
+	1650 3150 1650 3200
+Wire Wire Line
+	1900 3600 2150 3600
+Wire Wire Line
+	2550 2500 1650 2500
+Wire Wire Line
+	1650 2500 1650 3150
+Connection ~ 1650 3150
+Wire Wire Line
+	1650 3150 1250 3150
+$Comp
+L power:+5V #PWR?
+U 1 1 607AA896
+P 1950 4300
+F 0 "#PWR?" H 1950 4150 50  0001 C CNN
+F 1 "+5V" H 1965 4473 50  0000 C CNN
+F 2 "" H 1950 4300 50  0001 C CNN
+F 3 "" H 1950 4300 50  0001 C CNN
+	1    1950 4300
+	1    0    0    -1
+$EndComp
+Wire Wire Line
+	2550 4200 2550 4350
+Wire Wire Line
+	2550 4350 1950 4350
+Wire Wire Line
+	1250 4150 1250 4350
+Wire Wire Line
+	1950 4350 1950 4300
+Connection ~ 1950 4350
+Wire Wire Line
+	1950 4350 1250 4350
+$Comp
+L power:+5V #PWR?
+U 1 1 607ADABC
+P 1400 3450
+F 0 "#PWR?" H 1400 3300 50  0001 C CNN
+F 1 "+5V" H 1415 3623 50  0000 C CNN
+F 2 "" H 1400 3450 50  0001 C CNN
+F 3 "" H 1400 3450 50  0001 C CNN
+	1    1400 3450
+	1    0    0    -1
+$EndComp
+Wire Wire Line
+	1250 3150 1250 3850
+Wire Wire Line
+	1450 3700 1400 3700
+Wire Wire Line
+	1400 3700 1400 3450
 $EndSCHEMATC
